Commit message: Renamed all Nodes and thruster/arm controller to commander (and added _pkg)

File: src/arm_simulation/urdf/armsim.urdf.xacro (robot description, xacro)
@@ -14,14 +14,14 @@
       <origin xyz="0 0 0" rpy="0 0 0"/>
       <geometry>
-        <mesh filename="package://arm_controller/meshfiles/base_link.STL" />
-      </geometry>
-      <material name="light_blue">
-        <color rgba="0.792156862745098 0.819607843137255 0.933333333333333 1"/>
-      </material>
-    </visual>
-    <collision>
-      <origin xyz="0 0 0" rpy="0 0 0"/>
-      <geometry>
-        <mesh filename="package://arm_controller/meshfiles/base_link.STL"  />
+        <mesh filename="package://arm_commander/meshfiles/base_link.STL" />
+      </geometry>
+      <material name="light_blue">
+        <color rgba="0.792156862745098 0.819607843137255 0.933333333333333 1"/>
+      </material>
+    </visual>
+    <collision>
+      <origin xyz="0 0 0" rpy="0 0 0"/>
+      <geometry>
+        <mesh filename="package://arm_commander/meshfiles/base_link.STL"  />
       </geometry>
     </collision>
@@ -50,14 +50,14 @@
       <origin xyz="0 0 0" rpy="0 0 0"/>
       <geometry>
-        <mesh filename="package://arm_controller/meshfiles/Ax1.STL" />
-      </geometry>
-      <material name="light_blue">
-        <color rgba="0.792156862745098 0.819607843137255 0.933333333333333 1"/>
-      </material>
-    </visual>
-    <collision>
-      <origin xyz="0 0 0" rpy="0 0 0"/>
-      <geometry>
-        <mesh filename="package://arm_controller/meshfiles/Ax1.STL" />
+        <mesh filename="package://arm_commander/meshfiles/Ax1.STL" />
+      </geometry>
+      <material name="light_blue">
+        <color rgba="0.792156862745098 0.819607843137255 0.933333333333333 1"/>
+      </material>
+    </visual>
+    <collision>
+      <origin xyz="0 0 0" rpy="0 0 0"/>
+      <geometry>
+        <mesh filename="package://arm_commander/meshfiles/Ax1.STL" />
       </geometry>
     </collision>
@@ -85,14 +85,14 @@
       <origin xyz="0 0 0" rpy="0 0 0"/>
       <geometry>
-        <mesh filename="package://arm_controller/meshfiles/Ax2.STL" />
-      </geometry>
-      <material name="light_blue">
-        <color rgba="0.792156862745098 0.819607843137255 0.933333333333333 1"/>
-      </material>
-    </visual>
-    <collision>
-      <origin xyz="0 0 0" rpy="0 0 0"/>
-      <geometry>
-        <mesh filename="package://arm_controller/meshfiles/Ax2.STL" />
+        <mesh filename="package://arm_commander/meshfiles/Ax2.STL" />
+      </geometry>
+      <material name="light_blue">
+        <color rgba="0.792156862745098 0.819607843137255 0.933333333333333 1"/>
+      </material>
+    </visual>
+    <collision>
+      <origin xyz="0 0 0" rpy="0 0 0"/>
+      <geometry>
+        <mesh filename="package://arm_commander/meshfiles/Ax2.STL" />
       </geometry>
     </collision>
@@ -120,14 +120,14 @@
       <origin xyz="0 0 0" rpy="0 0 0"/>
       <geometry>
-        <mesh filename="package://arm_controller/meshfiles/Ax3.STL" />
-      </geometry>
-      <material name="light_blue">
-        <color rgba="0.792156862745098 0.819607843137255 0.933333333333333 1"/>
-      </material>
-    </visual>
-    <collision>
-      <origin xyz="0 0 0" rpy="0 0 0"/>
-      <geometry>
-        <mesh filename="package://arm_controller/meshfiles/Ax3.STL" />
+        <mesh filename="package://arm_commander/meshfiles/Ax3.STL" />
+      </geometry>
+      <material name="light_blue">
+        <color rgba="0.792156862745098 0.819607843137255 0.933333333333333 1"/>
+      </material>
+    </visual>
+    <collision>
+      <origin xyz="0 0 0" rpy="0 0 0"/>
+      <geometry>
+        <mesh filename="package://arm_commander/meshfiles/Ax3.STL" />
       </geometry>
     </collision>
@@ -156,5 +156,5 @@
       <origin xyz="0 0 0" rpy="0 0 0"/>
       <geometry>
-        <mesh filename="package://arm_controller/meshfiles/Ax4.STL"/>
+        <mesh filename="package://arm_commander/meshfiles/Ax4.STL"/>
       </geometry>
       <material name="grey">
@@ -165,5 +165,5 @@
       <origin xyz="0 0 0" rpy="0 0 0"/>
       <geometry>
-        <mesh filename="package://arm_controller/meshfiles/Ax4.STL"/>
+        <mesh filename="package://arm_commander/meshfiles/Ax4.STL"/>
       </geometry>
     </collision>
@@ -191,14 +191,14 @@
       <origin xyz="0 0 0" rpy="0 0 0"/>
       <geometry>
-        <mesh filename="package://arm_controller/meshfiles/Ax5.STL" />
-      </geometry>
-      <material name="light_blue">
-        <color rgba="0.792156862745098 0.819607843137255 0.933333333333333 1"/>
-      </material>
-    </visual>
-    <collision>
-      <origin xyz="0 0 0" rpy="0 0 0"/>
-      <geometry>
-        <mesh filename="package://arm_controller/meshfiles/Ax5.STL" />
+        <mesh filename="package://arm_commander/meshfiles/Ax5.STL" />
+      </geometry>
+      <material name="light_blue">
+        <color rgba="0.792156862745098 0.819607843137255 0.933333333333333 1"/>
+      </material>
+    </visual>
+    <collision>
+      <origin xyz="0 0 0" rpy="0 0 0"/>
+      <geometry>
+        <mesh filename="package://arm_commander/meshfiles/Ax5.STL" />
       </geometry>
     </collision>
